File: overboard.kicad_pcb (KiCad board)
At the start: 2 copper layers, 2.4 x 14.2 mm, 243 parts, among them J1 USB_C_Receptacle_USB2.0, J2 Trackpoint, K1 Key_Switch_LED, K10 Key_Switch_LED, K11 Key_Switch_LED, K12 Key_Switch_LED, K13 Key_Switch_LED, K14 Key_Switch_LED, K15 Key_Switch_LED, K16 Key_Switch_LED, K17 Key_Switch_LED, K18 Key_Switch_LED, K19 Key_Switch_LED, K2 Key_Switch_LED, K20 Key_Switch_LED, K21 Key_Switch_LED, K22 Key_Switch_LED, K23 Key_Switch_LED, K24 Key_Switch_LED, K25 Key_Switch_LED, K26 Key_Switch_LED, K27 Key_Switch_LED, K28 Key_Switch_LED, K29 Key_Switch_LED, K3 Key_Switch_LED, K30 Key_Switch_LED, K31 Key_Switch_LED, K32 Key_Switch_LED, K33 Key_Switch_LED, K34 Key_Switch_LED, K35 Key_Switch_LED, K36 Key_Switch_LED, K37 Key_Switch_LED, K38 Key_Switch_LED, K39 Key_Switch_LED, K4 Key_Switch_LED, K40 Key_Switch_LED, K41 Key_Switch_LED, K42 Key_Switch_LED, K43 Key_Switch_LED, K44 Key_Switch_LED, K45 Key_Switch_LED, K46 Key_Switch_LED, K47 Key_Switch_LED, K48 Key_Switch_LED, K49 Key_Switch, K5 Key_Switch_LED, K50 Key_Switch, K51 Key_Switch, K6 Key_Switch_LED, K7 Key_Switch_LED, K8 Key_Switch_LED, K9 Key_Switch_LED, Q1 Q_NMOS_DGS, Q2 Q_NPN_Darlington_BCE, Q3 Q_NPN_Darlington_BCE, SW1 SW_DIP_x04, SW2 RotaryEncoder_Switch, SW3 RotaryEncoder_Switch, SW4 SW_Push, U1 Teensy2.0++, U2 SKQUCAA010, U3 SKQUCAA010

Commit message: Changes
Parts:
- removed the SW1 at (33.3, 79.3)
- added D49: LED, LED_THT:LED_D1.8mm_W3.3mm_H2.4mm, F.Cu at (174.7, 174.9)
- added D50: LED, LED_THT:LED_D1.8mm_W3.3mm_H2.4mm, F.Cu at (210.1, 170.7)
- added D51: LED, LED_THT:LED_D1.8mm_W3.3mm_H2.4mm, F.Cu at (361.9, 70.0)
- added D52: LED, LED_THT:LED_D1.8mm_W3.3mm_H2.4mm, F.Cu at (186.5, 170.7)
- added D53: LED, LED_THT:LED_D1.8mm_W3.3mm_H2.4mm, F.Cu at (186.5, 174.9)
- added D54: LED, LED_THT:LED_D1.8mm_W3.3mm_H2.4mm, F.Cu at (347.7, 90.1)
- added D55: LED, LED_THT:LED_D1.8mm_W3.3mm_H2.4mm, F.Cu at (245.5, 174.9)
- added D56: LED, LED_THT:LED_D1.8mm_W3.3mm_H2.4mm, F.Cu at (204.2, 170.7)
- added D57: LED, LED_THT:LED_D1.8mm_W3.3mm_H2.4mm, F.Cu at (341.8, 90.1)
- added D58: LED, LED_THT:LED_D1.8mm_W3.3mm_H2.4mm, F.Cu at (239.6, 170.7)
- added D59: LED, LED_THT:LED_D1.8mm_W3.3mm_H2.4mm, F.Cu at (257.3, 170.7)
- added D60: LED, LED_THT:LED_D1.8mm_W3.3mm_H2.4mm, F.Cu at (257.3, 174.9)
- added D61: LED, LED_THT:LED_D1.8mm_W3.3mm_H2.4mm, F.Cu at (227.8, 170.7)
- added D62: LED, LED_THT:LED_D1.8mm_W3.3mm_H2.4mm, F.Cu at (356.1, 70.0)
- added D63: LED, LED_THT:LED_D1.8mm_W3.3mm_H2.4mm, F.Cu at (335.9, 90.1)
- added D64: LED, LED_THT:LED_D1.8mm_W3.3mm_H2.4mm, F.Cu at (361.9, 74.1)
- added D65: LED, LED_THT:LED_D1.8mm_W3.3mm_H2.4mm, F.Cu at (174.7, 170.7)
- added D66: LED, LED_THT:LED_D1.8mm_W3.3mm_H2.4mm, F.Cu at (356.1, 74.1)
- added D67: LED, LED_THT:LED_D1.8mm_W3.3mm_H2.4mm, F.Cu at (367.9, 70.0)
- added D68: LED, LED_THT:LED_D1.8mm_W3.3mm_H2.4mm, F.Cu at (335.9, 94.3)
- added D69: LED, LED_THT:LED_D1.8mm_W3.3mm_H2.4mm, F.Cu at (221.9, 174.9)
- added D70: LED, LED_THT:LED_D1.8mm_W3.3mm_H2.4mm, F.Cu at (233.7, 174.9)
- added D71: LED, LED_THT:LED_D1.8mm_W3.3mm_H2.4mm, F.Cu at (180.6, 170.7)
- added D72: LED, LED_THT:LED_D1.8mm_W3.3mm_H2.4mm, F.Cu at (251.4, 174.9)
- added D73: LED, LED_THT:LED_D1.8mm_W3.3mm_H2.4mm, F.Cu at (376.2, 58.1)
- added D74: LED, LED_THT:LED_D1.8mm_W3.3mm_H2.4mm, F.Cu at (192.4, 170.7)
- added D75: LED, LED_THT:LED_D1.8mm_W3.3mm_H2.4mm, F.Cu at (216.0, 174.9)
- added D76: LED, LED_THT:LED_D1.8mm_W3.3mm_H2.4mm, F.Cu at (216.0, 170.7)
- added D77: LED, LED_THT:LED_D1.8mm_W3.3mm_H2.4mm, F.Cu at (335.9, 98.4)
- added D78: LED, LED_THT:LED_D1.8mm_W3.3mm_H2.4mm, F.Cu at (382.1, 54.0)
- added D79: LED, LED_THT:LED_D1.8mm_W3.3mm_H2.4mm, F.Cu at (356.1, 78.3)
- added D80: LED, LED_THT:LED_D1.8mm_W3.3mm_H2.4mm, F.Cu at (376.2, 54.0)
- added D81: LED, LED_THT:LED_D1.8mm_W3.3mm_H2.4mm, F.Cu at (245.5, 170.7)
- added D82: LED, LED_THT:LED_D1.8mm_W3.3mm_H2.4mm, F.Cu at (221.9, 170.7)
- added D83: LED, LED_THT:LED_D1.8mm_W3.3mm_H2.4mm, F.Cu at (239.6, 174.9)
- added D84: LED, LED_THT:LED_D1.8mm_W3.3mm_H2.4mm, F.Cu at (210.1, 174.9)
- added D85: LED, LED_THT:LED_D1.8mm_W3.3mm_H2.4mm, F.Cu at (376.2, 49.8)
- added D86: LED, LED_THT:LED_D1.8mm_W3.3mm_H2.4mm, F.Cu at (227.8, 174.9)
- added D87: LED, LED_THT:LED_D1.8mm_W3.3mm_H2.4mm, F.Cu at (198.3, 174.9)
- added D88: LED, LED_THT:LED_D1.8mm_W3.3mm_H2.4mm, F.Cu at (180.6, 174.9)
- added D89: LED, LED_THT:LED_D1.8mm_W3.3mm_H2.4mm, F.Cu at (192.4, 174.9)
- added D90: LED, LED_THT:LED_D1.8mm_W3.3mm_H2.4mm, F.Cu at (204.2, 174.9)
- added D91: LED, LED_THT:LED_D1.8mm_W3.3mm_H2.4mm, F.Cu at (295.6, 150.6)
- added D92: LED, LED_THT:LED_D1.8mm_W3.3mm_H2.4mm, F.Cu at (233.7, 170.7)
- added D93: LED, LED_THT:LED_D1.8mm_W3.3mm_H2.4mm, F.Cu at (341.8, 94.3)
- added D94: LED, LED_THT:LED_D1.8mm_W3.3mm_H2.4mm, F.Cu at (382.1, 49.8)
- added D95: LED, LED_THT:LED_D1.8mm_W3.3mm_H2.4mm, F.Cu at (251.4, 170.7)
- added D96: LED, LED_THT:LED_D1.8mm_W3.3mm_H2.4mm, F.Cu at (198.3, 170.7)
- added J1: Pimoroni_Trackball, Kicad-Footprints:pimoroni_trackball, F.Cu at (25.9, 141.7)
- added S1: DS04-254-1L-02BK, DS04-254-1L-02BK:SW_DS04-254-1L-02BK, F.Cu at (52.9, 137.4)
- added S2: DS04-254-1L-02BK, DS04-254-1L-02BK:SW_DS04-254-1L-02BK, F.Cu at (52.9, 145.0)
- C1: footprint Capacitor_THT:CP_Radial_Tantal_D4.5mm_P2.50mm -> Capacitor_THT:CP_Radial_D5.0mm_P2.00mm
- J3: renamed from J1; footprint LED_THT:LED_D1.8mm_W3.3mm_H2.4mm -> Connector_USB:USB_C_Receptacle_HRO_TYPE-C-31-M-12
- K1, K10, K11, K12, K13, K14, K15, K16, K17, K18, K19, K2, K20, K21, K22, K23, K24, K25, K26, K27, K28, K29, K3, K30, K31, K32, K33, K34, K35, K36, K37, K38, K39, K4, K40, K41, K42, K43, K44, K45, K46, K47, K48, K5, K6, K7, K8, K9: value Key_Switch_LED -> Key_Switch; footprint LED_THT:LED_D1.8mm_W3.3mm_H2.4mm -> Switch_Keyboard_Hotswap_Kailh:SW_Hotswap_Kailh_MX_1.00u
- K49, K50, K51: footprint Switch_Keyboard_Hotswap_Kailh:SW_Hotswap_Kailh_MX_1.00u -> Button_Switch_Keyboard:SW_Cherry_MX_1.00u_PCB
- L1, L2: footprint Inductor_THT:L_Axial_L5.3mm_D2.2mm_P2.54mm_Vertical_Vishay_IM-1 -> Connector_JST:JST_PH_S2B-PH-SM4-TB_1x02-1MP_P2.00mm_Horizontal
- LCD1: footprint Keebio-Parts:Resistor -> Display_0xLib:OLED_I2C_128x64_0.96inch
- LS1, LS2: footprint Keebio-Parts:Resistor -> Buzzer_Beeper:Buzzer_Mallory_AST1109MLTRQ
- Q1, Q2, Q3: footprint Keebio-Parts:Resistor -> digikey-footprints:TO-220-3
- SW3: renamed from SW4; footprint Button_Switch_THT:SW_PUSH_6mm -> User:Bourns 7914H
- moved K45 241.2 mm to (344.3, 78.0)
- moved K17 238.4 mm to (324.1, 57.8)
- moved K10 227.6 mm to (364.4, 57.8)
- moved K16 217.3 mm to (324.1, 118.3)
- moved K39 207.3 mm to (304.0, 118.3)
- moved K8 203.7 mm to (304.0, 78.0)
- moved K28 197.4 mm to (324.1, 98.1)
- moved K48 187.4 mm to (304.0, 138.4)
- moved K43 174.9 mm to (263.7, 138.4)
- moved K2 173.2 mm to (283.9, 158.6)
- moved K32 172.7 mm to (324.1, 78.0)
- moved K35 172.5 mm to (304.0, 57.8)
- moved K9 172.4 mm to (283.9, 118.3)
- moved K11 167.9 mm to (344.3, 57.8)
- moved K23 156.7 mm to (263.7, 158.6)
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- renumbered D49 to D1, D58 to D10, D4 to D100, D5 to D101, D6 to D102, D7 to D103, D8 to D104, D9 to D105, D10 to D106, D11 to D107, D12 to D108, D13 to D109, D59 to D11, D14 to D110, D15 to D111, D16 to D112, D17 to D113, D18 to D114, D19 to D115, D20 to D116, D21 to D117, D22 to D118, D23 to D119, D60 to D12, D24 to D120, D25 to D121, D26 to D122, D27 to D123, D28 to D124, D29 to D125, D30 to D126, D31 to D127, D32 to D128, D33 to D129, D61 to D13, D34 to D130, D35 to D131, D36 to D132, D37 to D133, D38 to D134, D39 to D135, D40 to D136, D41 to D137, D42 to D138, D43 to D139, D62 to D14, D44 to D140, D45 to D141, D46 to D142, D47 to D143, D48 to D144, D99 to D145, D107 to D146, D102 to D147, D109 to D148, D97 to D149, D63 to D15, D98 to D150, D103 to D151, D104 to D152, D108 to D153, D100 to D154, D101 to D155, D105 to D156, D106 to D157, D110 to D158, D111 to D159, D64 to D16, D112 to D160, D113 to D161, D114 to D162, D115 to D163, D116 to D164, D117 to D165, D65 to D17, D66 to D18, D67 to D19, D50 to D2, D68 to D20, D69 to D21, D70 to D22, D71 to D23, D72 to D24, D73 to D25, D74 to D26, D75 to D27, D76 to D28, D77 to D29, D51 to D3, D78 to D30, D79 to D31, D80 to D32, D81 to D33, D82 to D34, D83 to D35, D84 to D36, D85 to D37, D86 to D38, D87 to D39, D52 to D4, D88 to D40, D89 to D41, D90 to D42, D91 to D43, D92 to D44, D93 to D45, D94 to D46, D95 to D47, D96 to D48, D53 to D5, D54 to D6, D55 to D7, D56 to D8, D57 to D9, D1 to D97, D2 to D98, D3 to D99, R15 to R1, R17 to R15, R18 to R16, R19 to R17, R20 to R18, R21 to R19, R16 to R2, R22 to R20, R23 to R21, R24 to R22, R25 to R23, R26 to R24, R27 to R25, R28 to R26, R29 to R27, R30 to R28, R31 to R29, R32 to R30, R33 to R31, R34 to R32, R35 to R33, R36 to R34, R37 to R35, R38 to R36, R39 to R37, R40 to R38, R41 to R39, R42 to R40, R43 to R41, R44 to R42, R45 to R43, R46 to R44, R47 to R45, R48 to R46, R49 to R47, R50 to R48, R51 to R49, R52 to R50, R55 to R51, R56 to R52, R57 to R53, R1 to R54, R2 to R55, R53 to R56, R54 to R57, SW2 to SW1, SW3 to SW2
Connections:
- K49 pad 1: COL9 -> COL7
- K50 pad 1: COL9 -> COL7
- K51 pad 1: COL9 -> COL7
- R54 pad 1: Net-(J1-PadA5) -> Net-(J3-PadA5)
- R55 pad 1: Net-(J1-PadB5) -> Net-(J3-PadB5)
- SW1 pad S1: COL9 -> COL7
- SW2 pad S1: COL9 -> COL7
- U2 pad 4: COL6 -> COL8
- U3 pad 4: COL8 -> COL9

Commit message: Add USB-C port
Parts:
- removed D1, D14, D145, D146, D147, D148, D149, D15, D150, D151, D152, D153, D154, D155, D156, D157, D158, D16, D161, D162, D163, D164, D165, D17, D18, D19, D2, D24, D25, D26, D27, D28, D29, D3, D34, D35, D36, D37, D38, D39, D4, D44, D45, D46, D47, D48, D5, D6, D7, D8, D9: 1N4148, Diode_THT:D_DO-35_SOD27_P7.62mm_Horizontal
- removed D100, D101, D102, D103, D104, D105, D106, D107, D108, D109, D110, D111, D112, D113, D114, D115, D116, D117, D118, D119, D120, D121, D122, D123, D124, D125, D126, D127, D128, D129, D130, D131, D132, D133, D134, D135, D136, D137, D138, D139, D140, D141, D142, D143, D144, D97, D98, D99: SK6812MINI-E, LED_SMD_0xLib:LED_SK6812MINI-E_3.2x2.8mm
- removed D159, D160: 1N4001, Diode_THT:D_DO-41_SOD81_P10.16mm_Horizontal
- removed D49, D54, D55, D56, D57, D58, D59, D65, D66, D67, D68, D69, D74, D75, D76, D77, D78, D79, D85, D86, D87, D88, D89, D95, D96: LED, LED_THT:LED_D1.8mm_W3.3mm_H2.4mm
- removed J3: USB_C_Receptacle_USB2.0, Connector_USB:USB_C_Receptacle_HRO_TYPE-C-31-M-12
- removed K1, K14, K15, K16, K17, K18, K19, K2, K24, K25, K26, K27, K28, K29, K3, K34, K35, K36, K37, K38, K39, K4, K44, K45, K46, K47, K48, K5, K6, K7, K8, K9: Key_Switch, Switch_Keyboard_Hotswap_Kailh:SW_Hotswap_Kailh_MX_1.00u
- removed K49: Key_Switch, Button_Switch_Keyboard:SW_Cherry_MX_1.00u_PCB
- removed LCD1: OLED_I2C, Display_0xLib:OLED_I2C_128x64_0.96inch
- removed LS2: AST1109MLTRQ, Buzzer_Beeper:Buzzer_Mallory_AST1109MLTRQ
- removed R13, R14, R15, R16, R17, R18, R19, R20, R21, R22, R23, R24, R25, R26, R27, R28, R29, R30, R31, R32, R33, R34, R35, R36, R37, R38, R39, R40, R41, R42, R43, R44, R45, R46, R47, R48, R49, R50: 470, Keebio-Parts:Resistor
- removed R51, R53: 4.7k, Keebio-Parts:Resistor
- removed R52: 100k, Keebio-Parts:Resistor
- removed R54, R55: 5.1k, Keebio-Parts:Resistor
- removed R56, R57: 1k, Keebio-Parts:Resistor
- removed S1, S2: DS04-254-1L-02BK, DS04-254-1L-02BK:SW_DS04-254-1L-02BK
- removed SW1, SW2: RotaryEncoder_Switch, Encoder:RollerEncoder_Panasonic_EVQWGD001
- removed SW3: SW_Push, User:Bourns 7914H
- removed U2, U3: SKQUCAA010, Alps SKQUCAA010:SKQUCAA010
- added D00: 1N4148, User:Diode_THT, F.Cu at (204.0, 25.8)
- added D01: 1N4148, User:Diode_THT, F.Cu at (384.5, -80.1)
- added D02: 1N4148, User:Diode_THT, F.Cu at (383.2, -90.7)
- added D03: 1N4148, User:Diode_THT, F.Cu at (373.8, -75.9)
- added DA0: 1N4148, User:Diode_THT, F.Cu at (337.9, -34.7)
- added DA1: 1N4148, User:Diode_THT, F.Cu at (346.5, -46.8)
- added DA2: 1N4148, User:Diode_THT, F.Cu at (366.7, -67.0)
- added DA3: 1N4148, User:Diode_THT, F.Cu at (383.2, -83.6)
- added DB0: 1N4148, User:Diode_THT, F.Cu at (232.4, -66.3)
- added DB1: 1N4148, User:Diode_THT, F.Cu at (373.8, -79.5)
- added DB2: 1N4148, User:Diode_THT, F.Cu at (366.7, -63.4)
- added DB3: 1N4148, User:Diode_THT, F.Cu at (325.2, -30.1)
- added DC0: 1N4148, User:Diode_THT, F.Cu at (383.2, -87.2)
- added DC1: 1N4148, User:Diode_THT, F.Cu at (366.7, -70.5)
- added DC2: 1N4148, User:Diode_THT, F.Cu at (284.8, 10.3)
- added DC3: 1N4148, User:Diode_THT, F.Cu at (284.8, 20.9)
- added DD0: 1N4148, User:Diode_THT, F.Cu at (295.6, 10.3)
- added DD1: 1N4148, User:Diode_THT, F.Cu at (325.2, -23.0)
- added DD2: 1N4148, User:Diode_THT, F.Cu at (346.5, -50.3)
- added DD3: 1N4148, User:Diode_THT, F.Cu at (284.8, 17.4)
- added DE0: 1N4148, User:Diode_THT, F.Cu at (327.1, -34.7)
- added DE1: 1N4148, User:Diode_THT, F.Cu at (325.2, -26.6)
- added DE2: 1N4148, User:Diode_THT, F.Cu at (336.0, -31.1)
- added DE3: 1N4148, User:Diode_THT, F.Cu at (284.8, 13.8)
- added DF0: 1N4148, User:Diode_THT, F.Cu at (305.0, 1.34)
- added DF1: 1N4148, User:Diode_THT, F.Cu at (346.5, -43.2)
- added DF2: 1N4148, User:Diode_THT, F.Cu at (358.1, -54.9)
- added DF3: 1N4148, User:Diode_THT, F.Cu at (347.3, -54.9)
- added DIP1: DS04-254-1L-04BK, DS04-254-1L-04BK:SW_DS04-254-1L-04BK, F.Cu at (228.6, 23.0)
- added DL1: 1N4001, Diode_THT:D_DO-41_SOD81_P7.62mm_Horizontal, F.Cu at (232.7, -70.2)
- added DL2: 1N4001, Diode_THT:D_DO-41_SOD81_P7.62mm_Horizontal, F.Cu at (204.3, 21.9)
- added ENC1: RotaryEncoder_Switch, User:Panasonic_EVQ-WGD001_LargerCutout, F.Cu at (334.6, -44.6)
- added ENC2: RotaryEncoder_Switch, User:Panasonic_EVQ-WGD001_LargerCutout, F.Cu at (354.8, -64.8)
- added H1: MountingHole, User:MountingHole_2.4mm_M2, F.Cu at (352.9, -28.9)
- added H2: MountingHole, User:MountingHole_2.4mm_M2, F.Cu at (411.0, -85.0)
- added H3: MountingHole, User:MountingHole_2.4mm_M2, F.Cu at (304.5, 20.7)
- added H4: MountingHole, User:MountingHole_2.4mm_M2, F.Cu at (344.9, -21.9)
- added H5: MountingHole, User:Trackpoint_Mounting_Holes, F.Cu at (213.5, -62.6)
- added K00: Key_Switch, MK_Switches:MXOnly-1U-NoLED, F.Cu at (215.1, -15.6)
- added K01: Key_Switch, MK_Switches:MXOnly-1U-NoLED, F.Cu at (237.2, -59.1)
- added K02: Key_Switch, MK_Switches:MXOnly-1U-NoLED, F.Cu at (297.8, -47.1)
- added K03: Key_Switch, MK_Switches:MXOnly-1U-NoLED, F.Cu at (215.1, -35.8)
- added K52: Key_Switch, MK_Switches:MXOnly-1U-NoLED, F.Cu at (215.1, 4.59)
- added K53: Key_Switch, MK_Switches:MXOnly-1U-NoLED, F.Cu at (295.9, -26.9)
- added K92: Key_Switch, MK_Switches:MXOnly-1U-NoLED, F.Cu at (215.1, -56.0)
- added K93: Key_Switch, MK_Switches:MXOnly-1U-NoLED, F.Cu at (263.6, -87.5)
- added K94: Key_Switch, MK_Switches:MXOnly-1U-NoLED, F.Cu at (257.4, -67.3)
- added KA0: Key_Switch, MK_Switches:MXOnly-1U-NoLED, F.Cu at (255.5, 13.5)
- added KA1: Key_Switch, MK_Switches:MXOnly-1U-NoLED, F.Cu at (277.6, -67.3)
- added KA2: Key_Switch, MK_Switches:MXOnly-1U-NoLED, F.Cu at (297.8, -67.3)
- added KA3: Key_Switch, MK_Switches:MXOnly-1U-NoLED, F.Cu at (318.0, -67.3)
- added KB0: Key_Switch, MK_Switches:MXOnly-1U-NoLED, F.Cu at (275.7, -6.67)
- added KB1: Key_Switch, MK_Switches:MXOnly-1U-NoLED, F.Cu at (304.0, -87.5)
- added KB2: Key_Switch, MK_Switches:MXOnly-1U-NoLED, F.Cu at (275.7, -26.9)
- added KB3: Key_Switch, MK_Switches:MXOnly-1U-NoLED, F.Cu at (344.4, -87.5)
- added KC0: Key_Switch, MK_Switches:MXOnly-1U-NoLED, F.Cu at (338.2, -67.3)
- added KC1: Key_Switch, MK_Switches:MXOnly-1U-NoLED, F.Cu at (324.2, -87.5)
- added KC2: Key_Switch, MK_Switches:MXOnly-1U-NoLED, F.Cu at (364.6, -87.5)
- added KC3: Key_Switch, MK_Switches:MXOnly-1U-NoLED, F.Cu at (316.1, -26.9)
- added KD0: Key_Switch, MK_Switches:MXOnly-1U-NoLED, F.Cu at (318.0, -47.1)
- added KD1: Key_Switch, MK_Switches:MXOnly-1U-NoLED, F.Cu at (257.4, -47.1)
- added KD2: Key_Switch, MK_Switches:MXOnly-1U-NoLED, F.Cu at (283.8, -87.5)
- added KD3: Key_Switch, MK_Switches:MXOnly-1U-NoLED, F.Cu at (295.9, -6.67)
- added KE0: Key_Switch, MK_Switches:MXOnly-1U-NoLED, F.Cu at (275.7, 13.5)
- added KE1: Key_Switch, MK_Switches:MXOnly-1U-NoLED, F.Cu at (255.5, -6.67)
- added KE2: Key_Switch, MK_Switches:MXOnly-1U-NoLED, F.Cu at (235.3, -38.9)
- added KE3: Key_Switch, MK_Switches:MXOnly-1U-NoLED, F.Cu at (243.4, -87.5)
- added KF0: Key_Switch, MK_Switches:MXOnly-1U-NoLED, F.Cu at (255.5, -26.9)
- added KF1: Key_Switch, MK_Switches:MXOnly-1U-NoLED, F.Cu at (277.6, -47.1)
- added KF2: Key_Switch, MK_Switches:MXOnly-1U-NoLED, F.Cu at (235.3, -18.7)
- added KF3: Key_Switch, MK_Switches:MXOnly-1U-NoLED, F.Cu at (235.3, 1.50)
- added LED1: LED, LED_THT:LED_D1.8mm_W3.3mm_H2.4mm, F.Cu at (373.5, -51.9)
- added LED2: LED, LED_THT:LED_D1.8mm_W3.3mm_H2.4mm, F.Cu at (403.4, -80.3)
- added LED3: LED, LED_THT:LED_D1.8mm_W3.3mm_H2.4mm, F.Cu at (218.0, 21.9)
- added NAV1: JOYSTICK_MINI, Sparkfun_Switches:JOYSTICK_MINI, F.Cu at (308.2, -6.06)
- added NAV2: JOYSTICK_MINI, Sparkfun_Switches:JOYSTICK_MINI, F.Cu at (376.9, -86.9)
- added OLED1: OLED_I2C, Display_0xLib:OLED_I2C_128x64_0.96inch, F.Cu at (45.2, 15.6)
- added RGB1: SK6812MINI-E, User:SK6812MINI-E_RGB_LED_3.2x2.8mm, F.Cu at (380.2, -61.5)
- added RGB10: SK6812MINI-E, User:SK6812MINI-E_RGB_LED_3.2x2.8mm, F.Cu at (238.1, 24.2)
- added RGB11: SK6812MINI-E, User:SK6812MINI-E_RGB_LED_3.2x2.8mm, F.Cu at (360.0, -50.6)
- added RGB12: SK6812MINI-E, User:SK6812MINI-E_RGB_LED_3.2x2.8mm, F.Cu at (335.9, -16.7)
- added RGB13: SK6812MINI-E, User:SK6812MINI-E_RGB_LED_3.2x2.8mm, F.Cu at (325.2, -8.61)
- added RGB14: SK6812MINI-E, User:SK6812MINI-E_RGB_LED_3.2x2.8mm, F.Cu at (327.9, -18.7)
- added RGB15: SK6812MINI-E, User:SK6812MINI-E_RGB_LED_3.2x2.8mm, F.Cu at (404.7, -90.0)
- added RGB16: SK6812MINI-E, User:SK6812MINI-E_RGB_LED_3.2x2.8mm, F.Cu at (306.3, 15.7)
- added RGB17: SK6812MINI-E, User:SK6812MINI-E_RGB_LED_3.2x2.8mm, F.Cu at (412.8, -90.0)
- added RGB18: SK6812MINI-E, User:SK6812MINI-E_RGB_LED_3.2x2.8mm, F.Cu at (335.9, -11.7)
- added RGB19: SK6812MINI-E, User:SK6812MINI-E_RGB_LED_3.2x2.8mm, F.Cu at (388.2, -70.7)
- added RGB2: SK6812MINI-E, User:SK6812MINI-E_RGB_LED_3.2x2.8mm, F.Cu at (307.7, 5.64)
- added RGB20: SK6812MINI-E, User:SK6812MINI-E_RGB_LED_3.2x2.8mm, F.Cu at (217.4, 26.6)
- added RGB21: SK6812MINI-E, User:SK6812MINI-E_RGB_LED_3.2x2.8mm, F.Cu at (309.0, 10.7)
- added RGB22: SK6812MINI-E, User:SK6812MINI-E_RGB_LED_3.2x2.8mm, F.Cu at (317.2, -4.11)
- added RGB23: SK6812MINI-E, User:SK6812MINI-E_RGB_LED_3.2x2.8mm, F.Cu at (380.2, -66.6)
- added RGB24: SK6812MINI-E, User:SK6812MINI-E_RGB_LED_3.2x2.8mm, F.Cu at (388.2, -65.7)
- added RGB25: SK6812MINI-E, User:SK6812MINI-E_RGB_LED_3.2x2.8mm, F.Cu at (368.0, -50.6)
- added RGB26: SK6812MINI-E, User:SK6812MINI-E_RGB_LED_3.2x2.8mm, F.Cu at (351.3, -38.9)
- added RGB27: SK6812MINI-E, User:SK6812MINI-E_RGB_LED_3.2x2.8mm, F.Cu at (398.0, -79.9)
- added RGB28: SK6812MINI-E, User:SK6812MINI-E_RGB_LED_3.2x2.8mm, F.Cu at (396.3, -74.8)
- added RGB29: SK6812MINI-E, User:SK6812MINI-E_RGB_LED_3.2x2.8mm, F.Cu at (346.7, -26.8)
- added RGB3: SK6812MINI-E, User:SK6812MINI-E_RGB_LED_3.2x2.8mm, F.Cu at (360.0, -40.5)
- added RGB30: SK6812MINI-E, User:SK6812MINI-E_RGB_LED_3.2x2.8mm, F.Cu at (371.5, -56.5)
- added RGB31: SK6812MINI-E, User:SK6812MINI-E_RGB_LED_3.2x2.8mm, F.Cu at (344.0, -16.7)
- added RGB32: SK6812MINI-E, User:SK6812MINI-E_RGB_LED_3.2x2.8mm, F.Cu at (298.2, 19.6)
- added RGB33: SK6812MINI-E, User:SK6812MINI-E_RGB_LED_3.2x2.8mm, F.Cu at (396.7, -84.9)
- added RGB34: SK6812MINI-E, User:SK6812MINI-E_RGB_LED_3.2x2.8mm, F.Cu at (326.5, -3.56)
- added RGB35: SK6812MINI-E, User:SK6812MINI-E_RGB_LED_3.2x2.8mm, F.Cu at (360.0, -45.5)
- added RGB36: SK6812MINI-E, User:SK6812MINI-E_RGB_LED_3.2x2.8mm, F.Cu at (404.7, -84.9)
- added RGB37: SK6812MINI-E, User:SK6812MINI-E_RGB_LED_3.2x2.8mm, F.Cu at (338.6, -26.8)
- added RGB38: SK6812MINI-E, User:SK6812MINI-E_RGB_LED_3.2x2.8mm, F.Cu at (388.2, -75.8)
- added RGB39: SK6812MINI-E, User:SK6812MINI-E_RGB_LED_3.2x2.8mm, F.Cu at (318.4, 0.94)
- added RGB4: SK6812MINI-E, User:SK6812MINI-E_RGB_LED_3.2x2.8mm, F.Cu at (287.5, 25.2)
- added RGB40: SK6812MINI-E, User:SK6812MINI-E_RGB_LED_3.2x2.8mm, F.Cu at (396.7, -90.0)
- added RGB41: SK6812MINI-E, User:SK6812MINI-E_RGB_LED_3.2x2.8mm, F.Cu at (327.9, -13.7)
- added RGB42: SK6812MINI-E, User:SK6812MINI-E_RGB_LED_3.2x2.8mm, F.Cu at (380.2, -71.6)
- added RGB43: SK6812MINI-E, User:SK6812MINI-E_RGB_LED_3.2x2.8mm, F.Cu at (338.6, -21.8)
- added RGB44: SK6812MINI-E, User:SK6812MINI-E_RGB_LED_3.2x2.8mm, F.Cu at (396.3, -69.8)
- added RGB45: SK6812MINI-E, User:SK6812MINI-E_RGB_LED_3.2x2.8mm, F.Cu at (298.2, 14.6)
- added RGB46: SK6812MINI-E, User:SK6812MINI-E_RGB_LED_3.2x2.8mm, F.Cu at (295.5, 25.2)
- added RGB47: SK6812MINI-E, User:SK6812MINI-E_RGB_LED_3.2x2.8mm, F.Cu at (317.1, 5.99)
- added RGB48: SK6812MINI-E, User:SK6812MINI-E_RGB_LED_3.2x2.8mm, F.Cu at (351.3, -33.9)
- added RGB5: SK6812MINI-E, User:SK6812MINI-E_RGB_LED_3.2x2.8mm, F.Cu at (368.0, -45.5)
- added RGB6: SK6812MINI-E, User:SK6812MINI-E_RGB_LED_3.2x2.8mm, F.Cu at (238.1, 19.2)
- added RGB7: SK6812MINI-E, User:SK6812MINI-E_RGB_LED_3.2x2.8mm, F.Cu at (379.6, -56.5)
- added RGB8: SK6812MINI-E, User:SK6812MINI-E_RGB_LED_3.2x2.8mm, F.Cu at (359.4, -35.4)
- added RGB9: SK6812MINI-E, User:SK6812MINI-E_RGB_LED_3.2x2.8mm, F.Cu at (317.2, -9.16)
- C1: footprint Capacitor_THT:CP_Radial_D5.0mm_P2.00mm -> Capacitor_THT:C_Radial_D4.0mm_H7.0mm_P1.50mm
- D10, D11, D12, D13, D20, D21, D22, D23, D30, D31, D32, D33, D40, D41, D42, D43: footprint Diode_THT:D_DO-35_SOD27_P7.62mm_Horizontal -> User:Diode_THT
- D50, D51, D52, D53, D90, D91, D92, D93, D94: value LED -> 1N4148; footprint LED_THT:LED_D1.8mm_W3.3mm_H2.4mm -> User:Diode_THT
- D60, D61, D62, D63, D64, D70, D71, D72, D73, D80, D81, D82, D83, D84: value LED -> 1N4148; footprint LED_THT:LED_D1.8mm_W3.3mm_H2.4mm -> Diode_SMD:D_SOD-123
- J1: value Pimoroni_Trackball -> USB_C_Receptacle_USB2.0; footprint Kicad-Footprints:pimoroni_trackball -> USB_Type-C:USB_C_Receptacle_HRO_TYPE-C-31-M-12
- J2: footprint pierce:TRACKPOINT -> Connector_PinHeader_2.54mm:PinHeader_1x05_P2.54mm_Vertical
- K10, K11, K12, K13, K20, K21, K22, K23, K30, K31, K32, K33, K40, K41, K42, K43: footprint Switch_Keyboard_Hotswap_Kailh:SW_Hotswap_Kailh_MX_1.00u -> MK_Switches:MXOnly-1U-NoLED
- K50, K51: footprint Button_Switch_Keyboard:SW_Cherry_MX_1.00u_PCB -> MK_Switches:MXOnly-1U-NoLED
- L1, L2: footprint Connector_JST:JST_PH_S2B-PH-SM4-TB_1x02-1MP_P2.00mm_Horizontal -> Connector_JST:JST_PH_S2B-PH-K_1x02_P2.00mm_Horizontal
- Q1: value Q_NMOS_DGS -> Q_NPN_Darlington_BCE
- Q3: value Q_NPN_Darlington_BCE -> Q_NMOS_DGS
- R1: value 10k -> 5.1k
- R2: value 470 -> 5.1k
- R3, R4: value 470 -> 4.7k
- R5: value 470 -> 100k
- R6, R7: value 470 -> 1k
- R8: value 470 -> 10k
- moved R11 77.9 mm to (98.4, 137.4)
- moved R12 69.6 mm to (98.4, 140.5)
- moved J2 33.4 mm to (89.7, 138.1)
Connections:
- D11 pad 1: ROW0 -> ROW1
- D12 pad 1: ROW0 -> ROW2
- D13 pad 1: ROW1 -> ROW3
- D20 pad 1: ROW1 -> ROW0
- D22 pad 1: ROW1 -> ROW2
- D23 pad 1: ROW1 -> ROW3
- D30 pad 1: ROW2 -> ROW0
- D31 pad 1: ROW2 -> ROW1
- D33 pad 1: ROW2 -> ROW3
- D40 pad 1: ROW3 -> ROW0
- D41 pad 1: ROW3 -> ROW1
- D42 pad 1: ROW3 -> ROW2
- D50 pad 1: Net-(D50-Pad1) -> ROW0
- D50 pad 2: VCC -> Net-(D50-Pad2)
- D51 pad 1: Net-(D51-Pad1) -> ROW1
- D51 pad 2: VCC -> Net-(D51-Pad2)
- D52 pad 1: Net-(D52-Pad1) -> ROW2
- D52 pad 2: VCC -> Net-(D52-Pad2)
- D53 pad 1: Net-(D53-Pad1) -> ROW3
- D53 pad 2: VCC -> Net-(D53-Pad2)
- D60 pad 1: Net-(D60-Pad1) -> ROW0
- D60 pad 2: VCC -> Net-(D60-Pad2)
- D61 pad 1: Net-(D61-Pad1) -> ROW1
- D61 pad 2: VCC -> Net-(D61-Pad2)
- D62 pad 1: Net-(D62-Pad1) -> ROW2
- D62 pad 2: VCC -> Net-(D62-Pad2)
- D63 pad 1: Net-(D63-Pad1) -> ROW3
- D63 pad 2: VCC -> Net-(D63-Pad2)
- D64 pad 1: Net-(D64-Pad1) -> ROW4
- D64 pad 2: VCC -> Net-(D64-Pad2)
- D70 pad 1: Net-(D70-Pad1) -> ROW0
- D70 pad 2: VCC -> Net-(D70-Pad2)
- D71 pad 1: Net-(D71-Pad1) -> ROW1
- D71 pad 2: VCC -> Net-(D71-Pad2)
- D72 pad 1: Net-(D72-Pad1) -> ROW2
- D72 pad 2: VCC -> Net-(D72-Pad2)
- D73 pad 1: Net-(D73-Pad1) -> ROW3
- D73 pad 2: VCC -> Net-(D73-Pad2)
- D80 pad 1: Net-(D80-Pad1) -> ROW0
- D80 pad 2: VCC -> Net-(D80-Pad2)
- D81 pad 1: Net-(D81-Pad1) -> ROW1
- D81 pad 2: VCC -> Net-(D81-Pad2)
- D82 pad 1: Net-(D82-Pad1) -> ROW2
- D82 pad 2: VCC -> Net-(D82-Pad2)
- D83 pad 1: Net-(D83-Pad1) -> ROW3
- D83 pad 2: VCC -> Net-(D83-Pad2)
- D84 pad 1: Net-(D84-Pad1) -> ROW4
- D84 pad 2: VCC -> Net-(D84-Pad2)
- D90 pad 1: Net-(D90-Pad1) -> ROW0
- D90 pad 2: VCC -> Net-(D90-Pad2)
- D91 pad 1: Net-(D91-Pad1) -> ROW1
- D91 pad 2: VCC -> Net-(D91-Pad2)
- D92 pad 1: Net-(D92-Pad1) -> ROW2
- D92 pad 2: VCC -> Net-(D92-Pad2)
- D93 pad 1: Net-(D93-Pad1) -> ROW3
- D93 pad 2: VCC -> Net-(D93-Pad2)
- D94 pad 1: Net-(D94-Pad1) -> ROW4
- D94 pad 2: VCC -> Net-(D94-Pad2)
- K10 pad 1: COL13 -> COL1
- K11 pad 1: COL14 -> COL1
- K12 pad 1: COL15 -> COL1
- K13 pad 1: COL0 -> COL1
- K20 pad 1: COL11 -> COL2
- K21 pad 1: COL12 -> COL2
- K22 pad 1: COL13 -> COL2
- K23 pad 1: COL14 -> COL2
- K30 pad 1: COL5 -> COL3
- K31 pad 1: COL10 -> COL3
- K32 pad 1: COL11 -> COL3
- K33 pad 1: COL12 -> COL3
- K40 pad 1: COL3 -> COL4
- K42 pad 1: COL5 -> COL4
- K43 pad 1: COL10 -> COL4
- K50 pad 1: COL7 -> COL5
- K50 pad 2: Net-(D164-Pad2) -> Net-(D50-Pad2)
- K51 pad 1: COL7 -> COL5
- K51 pad 2: Net-(D165-Pad2) -> Net-(D51-Pad2)
- L1 pad 1: Net-(D159-Pad2) -> Net-(DL1-Pad2)
- L2 pad 1: Net-(D160-Pad2) -> Net-(DL2-Pad2)
- Q1 pad 2: Net-(Q1-Pad2) -> Net-(DL1-Pad2)
- Q2 pad 2: Net-(D159-Pad2) -> Net-(DL2-Pad2)
- Q3 pad 2: Net-(D160-Pad2) -> Net-(Q3-Pad2)
- R1 pad 2: Net-(Q1-Pad2) -> Net-(J1-PadA5)
- R10 pad 2: Net-(Q1-Pad1) -> Net-(Q3-Pad1)
- R11 pad 2: Net-(Q1-Pad1) -> Net-(Q3-Pad1)
- R12 pad 2: Net-(Q1-Pad1) -> Net-(Q3-Pad1)
- R2 pad 1: Net-(Q1-Pad2) -> GND
- R2 pad 2: BACKLIGHT -> Net-(J1-PadB5)
- R3 pad 1: Net-(D49-Pad1) -> VCC
- R3 pad 2: Net-(Q1-Pad1) -> PS2_CLOCK
- R4 pad 1: Net-(D50-Pad1) -> VCC
- R4 pad 2: Net-(Q1-Pad1) -> PS2_DATA
- R5 pad 1: Net-(D51-Pad1) -> GND
- R5 pad 2: Net-(Q1-Pad1) -> Net-(C1-Pad2)
- R6 pad 1: Net-(D52-Pad1) -> SOLENOID1
- R7 pad 1: Net-(D53-Pad1) -> SOLENOID2
- R7 pad 2: Net-(Q1-Pad1) -> Net-(Q2-Pad1)
- R8 pad 1: Net-(D54-Pad1) -> GND
- R8 pad 2: Net-(Q1-Pad1) -> Net-(Q3-Pad2)
- R9 pad 1: Net-(D55-Pad1) -> Net-(Q3-Pad2)
- R9 pad 2: Net-(Q1-Pad1) -> BACKLIGHT
- U1 pad 10: ROW1 -> unconnected-(U1-Pad10)
- U1 pad 11: ROW2 -> unconnected-(U1-Pad11)
- U1 pad 12: ROW3 -> unconnected-(U1-Pad12)
- U1 pad 13: ROW4 -> unconnected-(U1-Pad13)
- U1 pad 14: ENC_A -> unconnected-(U1-Pad14)
- U1 pad 15: ENC_B1 -> unconnected-(U1-Pad15)
- U1 pad 16: ENC_B2 -> unconnected-(U1-Pad16)
- U1 pad 17: AUDIO -> SOLENOID2
- U1 pad 18: SOLENOID2 -> BACKLIGHT
- U1 pad 19: BACKLIGHT -> AUDIO
- U1 pad 2: AUDIO_ALT -> SOLENOID1
- U1 pad 20: RGB_DI -> unconnected-(U1-Pad20)
- U1 pad 24: COL15 -> unconnected-(U1-Pad24)
- U1 pad 25: COL14 -> unconnected-(U1-Pad25)
- U1 pad 26: COL13 -> unconnected-(U1-Pad26)
- U1 pad 27: COL12 -> unconnected-(U1-Pad27)
- U1 pad 28: COL11 -> unconnected-(U1-Pad28)
- U1 pad 29: COL10 -> unconnected-(U1-Pad29)
- U1 pad 30: COL9 -> unconnected-(U1-Pad30)
- U1 pad 31: COL8 -> unconnected-(U1-Pad31)
- U1 pad 34: COL7 -> unconnected-(U1-Pad34)
- U1 pad 35: COL6 -> unconnected-(U1-Pad35)
- U1 pad 36: COL5 -> unconnected-(U1-Pad36)
- U1 pad 37: COL4 -> unconnected-(U1-Pad37)
- U1 pad 38: COL3 -> unconnected-(U1-Pad38)
- U1 pad 39: COL2 -> unconnected-(U1-Pad39)
- U1 pad 40: COL1 -> unconnected-(U1-Pad40)
- U1 pad 41: COL0 -> unconnected-(U1-Pad41)
- U1 pad 42: SOLENOID -> RGB_DI
- U1 pad 9: ROW0 -> unconnected-(U1-Pad9)
Other:
- board size 2.4 x 14.2 mm -> 2.8 x 14.2 mm

Commit message: 48 switch layout
Parts:
- moved K10 479.5 mm to (-106.8, -30.6), turned to 173 degrees
- moved K11 458.7 mm to (-109.1, -11.7), turned to 173 degrees
- moved D02 432.5 mm to (-19.1, 68.1)
- moved D03 432.5 mm to (-28.6, 82.9)
- moved DA0 432.5 mm to (-64.4, 124.1)
- moved DA2 432.5 mm to (-35.6, 91.9)
- moved DA3 432.5 mm to (-19.1, 75.2)
- moved DB1 432.5 mm to (-28.6, 79.4)
- moved DB2 432.5 mm to (-35.6, 95.4)
- moved DC0 432.5 mm to (-19.1, 71.7)
- moved DC1 432.5 mm to (-35.6, 88.3)
- moved DC2 432.5 mm to (-117.5, 169.1)
- moved DC3 432.5 mm to (-117.5, 179.8)
- moved DD0 432.5 mm to (-106.7, 169.1)
- moved DD3 432.5 mm to (-117.5, 176.2)
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
Commit message: Add plate, place RGB LEDs
Parts:
- removed D60, D61, D62, D63, D64, D70, D71, D72, D73, D80, D81, D82, D83, D84: 1N4148, Diode_SMD:D_SOD-123
- removed DIP1: DS04-254-1L-04BK, DS04-254-1L-04BK:SW_DS04-254-1L-04BK
- removed H1, H2, H3, H4: MountingHole, User:MountingHole_2.4mm_M2
- removed H5: MountingHole, User:Trackpoint_Mounting_Holes
- removed NAV1, NAV2: JOYSTICK_MINI, Sparkfun_Switches:JOYSTICK_MINI
- added J3: Trackpoint, Connector_PinHeader_2.54mm:PinHeader_1x05_P2.54mm_Vertical, F.Cu at (-122.2, 66.7)
- added J4: Conn_01x02, Connector_PinHeader_2.54mm:PinHeader_1x02_P2.54mm_Vertical, F.Cu at (-117.6, 66.7)
- added J5: Conn_01x02, Connector_PinHeader_2.54mm:PinHeader_1x02_P2.54mm_Vertical, F.Cu at (-117.6, 73.9)
- added J6: Conn_01x02, Connector_PinHeader_2.54mm:PinHeader_1x02_P2.54mm_Vertical, F.Cu at (-108.3, 66.7)
- added J7: Conn_01x02, Connector_PinHeader_2.54mm:PinHeader_1x02_P2.54mm_Vertical, F.Cu at (-112.9, 66.7)
- added REF**: 60_PCB_Solenoid_Cutouts, User:60_PCB_Solenoid_Cutouts, F.Cu at (0.00, 0.00)
- added SW1: Reset_SW, User:Panasonic_EVPAW, F.Cu at (-112.2, 73.3)
- J1: value USB_C_Receptacle_USB2.0 -> HRO-TYPE-C-31-M-12; footprint USB_Type-C:USB_C_Receptacle_HRO_TYPE-C-31-M-12 -> Type-C:HRO-TYPE-C-31-M-12-HandSoldering
- J2: value Trackpoint -> Conn_01x04; footprint Connector_PinHeader_2.54mm:PinHeader_1x05_P2.54mm_Vertical -> Connector_PinSocket_2.54mm:PinSocket_1x04_P2.54mm_Vertical
- RGB1, RGB10, RGB11, RGB12, RGB13, RGB14, RGB15, RGB16, RGB17, RGB18, RGB19, RGB2, RGB20, RGB21, RGB22, RGB23, RGB24, RGB25, RGB26, RGB27, RGB28, RGB29, RGB3, RGB30, RGB31, RGB32, RGB33, RGB34, RGB35, RGB36, RGB37, RGB38, RGB39, RGB4, RGB40, RGB41, RGB42, RGB43, RGB44, RGB45, RGB46, RGB47, RGB48, RGB5, RGB6, RGB7, RGB8, RGB9: moved to B.Cu
- moved RGB4 296.8 mm to (87.3, -33.3), turned to -173 degrees
- moved RGB16 253.5 mm to (91.9, 4.48), turned to -173 degrees
- moved RGB6 246.3 mm to (125.1, -38.0), turned to -173 degrees
- moved RGB18 245.3 mm to (129.7, -0.16), turned to -173 degrees
- moved RGB2 241.0 mm to (49.5, -28.7), turned to -173 degrees
- moved RGB9 239.7 mm to (89.6, -14.4), turned to -173 degrees
- moved RGB21 237.8 mm to (94.3, 23.4), turned to -173 degrees
- moved RGB46 218.5 mm to (-68.4, -31.0), turned to 173 degrees
- moved RGB20 211.3 mm to (113.2, 21.1), turned to -173 degrees
- moved RGB45 207.4 mm to (-87.3, -33.3), turned to 173 degrees
- moved RGB8 206.3 mm to (108.5, -16.7), turned to -173 degrees
- moved RGB22 205.9 mm to (75.3, 25.7), turned to -173 degrees
- moved RGB5 204.7 mm to (106.2, -35.7), turned to -173 degrees
- moved RGB10 201.4 mm to (70.7, -12.1), turned to -173 degrees
- moved U1 198.1 mm to (0.00, -38.1)
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Connections:
- J2 pad 1: VCC -> VBUS
- J2 pad 2: GND -> D-
- J2 pad 3: PS2_CLOCK -> D+
- J2 pad 4: Net-(C1-Pad2) -> GND
- R1 pad 2: Net-(J1-PadA5) -> Net-(J1-Pad4)
- R2 pad 2: Net-(J1-PadB5) -> Net-(J1-Pad10)
Other:
- board size 2.8 x 14.2 mm -> 285 x 95.1 mm

Commit message: Place diodes
Parts:
- D00, D01, D02, D03, D10, D11, D12, D13, D20, D21, D22, D23, D30, D31, D32, D33, D40, D41, D42, D43, D50, D51, D52, D53, DA0, DA1, DA2, DA3, DB0, DB1, DB2, DB3, DC0, DC1, DC2, DC3, DD0, DD1, DD2, DD3, DE0, DE1, DE2, DE3, DF0, DF1, DF2, DF3: moved to B.Cu
- moved DF0 300.4 mm to (124.6, -42.4), turned to -173 degrees
- moved DD0 283.2 mm to (86.7, -37.7), turned to -173 degrees
- moved DE3 278.0 mm to (112.6, 16.7), turned to -173 degrees
- moved DD3 263.3 mm to (93.7, 19.0), turned to -173 degrees
- moved DC2 252.8 mm to (72.5, 2.39), turned to -173 degrees
- moved DC3 249.2 mm to (74.8, 21.3), turned to -173 degrees
- moved DE0 244.3 mm to (105.7, -40.1), turned to -173 degrees
- moved DE1 240.4 mm to (108.0, -21.2), turned to -173 degrees
- moved D13 236.0 mm to (-112.6, 16.7), turned to 173 degrees
- moved DF1 229.6 mm to (126.9, -23.5), turned to -173 degrees
- moved D00 229.1 mm to (-124.6, -42.4), turned to 173 degrees
- moved D50 228.8 mm to (-30.0, -30.8), turned to 173 degrees
- moved D22 228.2 mm to (-91.4, 0.07), turned to 173 degrees
- moved DD1 227.0 mm to (89.1, -18.8), turned to -173 degrees
- moved DE2 219.3 mm to (110.3, -2.25), turned to -173 degrees
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
Commit message: Place components
Parts:
- removed J6, J7: Conn_01x02, Connector_PinHeader_2.54mm:PinHeader_1x02_P2.54mm_Vertical
- added H1: G***, User:Trackpoint_Outline, F.Cu at (0.00, 2.60)
- C1, DL1, DL2, J1, SW1: moved to B.Cu
- D00, D01, D02, D03, D10, D11, D12, D13, D20, D21, D22, D23, D30, D31, D32, D33, D40, D41, D42, D43, D50, D51, D52, D53, DA0, DA1, DA2, DA3, DB0, DB1, DB2, DB3, DC0, DC1, DC2, DC3, DD0, DD1, DD2, DD3, DE0, DE1, DE2, DE3, DF0, DF1, DF2, DF3: footprint User:Diode_THT -> User:Diode_THT_P7.62mm
- D90, D91, D92, D93, D94: footprint User:Diode_THT -> User:Diode_THT_P7.62mm; moved to B.Cu
- J2: footprint Connector_PinSocket_2.54mm:PinSocket_1x04_P2.54mm_Vertical -> Connector_PinHeader_2.54mm:PinHeader_1x04_P2.54mm_Horizontal; moved to B.Cu
- J3: footprint Connector_PinHeader_2.54mm:PinHeader_1x05_P2.54mm_Vertical -> Connector_PinHeader_2.54mm:PinHeader_1x05_P2.54mm_Horizontal; moved to B.Cu
- J4, J5: value Conn_01x02 -> Conn_01x04; footprint Connector_PinHeader_2.54mm:PinHeader_1x02_P2.54mm_Vertical -> User:PinHeader_1x04_P2.54mm_Vertical_Centered
- K00, K01, K02, K03, K10, K11, K12, K13, K20, K21, K22, K23, K30, K31, K32, K33, K40, K41, K42, K43, K50, K51, K52, K53, K92, K93, K94, KA0, KA1, KA2, KA3, KB0, KB1, KB2, KB3, KC0, KC1, KC2, KC3, KD0, KD1, KD2, KD3, KE0, KE1, KE2, KE3, KF0, KF1, KF2, KF3: footprint MK_Switches:MXOnly-1U-NoLED -> User:MXOnly-1U
- L1, L2: footprint Connector_JST:JST_PH_S2B-PH-K_1x02_P2.00mm_Horizontal -> User:JST_PH_S2B-PH-K_1x02_P2.00mm_Horizontal; moved to B.Cu
- LED1, LED2, LED3: footprint LED_THT:LED_D1.8mm_W3.3mm_H2.4mm -> User:LED_D1.8mm_W3.3mm_H2.4mm
- OLED1: footprint Display_0xLib:OLED_I2C_128x64_0.96inch -> User:128x64OLED
- Q1, Q2, Q3: footprint digikey-footprints:TO-220-3 -> User:TO-220-3; moved to B.Cu
- R1, R10, R11, R12, R2, R3, R4, R5, R6, R7, R8, R9: footprint Keebio-Parts:Resistor -> User:Resistor_THT_P7.62mm; moved to B.Cu
- U1: footprint teensy:Teensy2.0++ -> User:Teensy2.0++_43Pin; moved to B.Cu
- moved J5 273.5 mm to (138.5, -22.2)
- moved RGB19 264.1 mm to (-132.1, 18.7), turned to -7 degrees
- moved RGB30 264.1 mm to (132.1, 18.7), turned to 7 degrees
- moved RGB18 259.5 mm to (-129.7, -0.16), turned to 173 degrees
- moved RGB31 259.5 mm to (129.7, -0.16), turned to -173 degrees
- moved RGB42 254.8 mm to (127.4, -19.1), turned to 7 degrees
- moved RGB7 254.8 mm to (-127.4, -19.1), turned to -7 degrees
- moved RGB43 250.2 mm to (125.1, -38.0), turned to -173 degrees
- moved RGB6 250.2 mm to (-125.1, -38.0), turned to 173 degrees
- moved J1 243.2 mm to (-124.3, -49.6)
- moved RGB20 226.3 mm to (-113.2, 21.1), turned to -7 degrees
- moved RGB29 226.3 mm to (113.2, 21.1), turned to 7 degrees
- moved R1 223.4 mm to (-136.3, -45.2)
- moved RGB17 221.7 mm to (-110.8, 2.16), turned to 173 degrees
- moved RGB32 221.7 mm to (110.8, 2.16), turned to -173 degrees
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Connections:
- J4 pad 2: COL6 -> ROW2
- J5 pad 1: ROW2 -> ROW1
- J5 pad 2: COL7 -> ROW3
- R10 pad 1: Net-(LED3-Pad1) -> Net-(LED1-Pad1)
- R12 pad 1: Net-(LED1-Pad1) -> Net-(LED3-Pad1)
Routing:
- added copper zone on B.Cu, net GND
- added copper zone on F.Cu, net GND
Other:
- outline, holes or cut-outs redrawn

Commit message: Route PCB & plate
Parts:
- DL1, DL2: footprint Diode_THT:D_DO-41_SOD81_P7.62mm_Horizontal -> User:1N4001
- moved DL1 107.9 mm to (-103.2, 17.8), turned to -97 degrees
- moved DL2 103.7 mm to (103.2, 17.8), turned to -83 degrees
- moved Q1 3.57 mm to (-15.4, -41.3)
- moved Q2 3.57 mm to (15.4, -41.3)
- moved LS1 3.57 mm to (27.0, -41.3)
- turned R6 to 0 degrees
- turned R7 to 180 degrees
Connections:
- U1 pad 10: unconnected-(U1-Pad10) -> ENC_B2
- U1 pad 11: unconnected-(U1-Pad11) -> COL9
- U1 pad 12: unconnected-(U1-Pad12) -> COL6
- U1 pad 13: unconnected-(U1-Pad13) -> COL7
- U1 pad 14: unconnected-(U1-Pad14) -> ROW0
- U1 pad 15: unconnected-(U1-Pad15) -> ROW1
- U1 pad 16: unconnected-(U1-Pad16) -> ROW4
- U1 pad 20: unconnected-(U1-Pad20) -> COL8
- U1 pad 24: unconnected-(U1-Pad24) -> COLA
- U1 pad 25: unconnected-(U1-Pad25) -> COLB
- U1 pad 26: unconnected-(U1-Pad26) -> COLC
- U1 pad 27: unconnected-(U1-Pad27) -> COLD
- U1 pad 28: unconnected-(U1-Pad28) -> COLE
- U1 pad 29: unconnected-(U1-Pad29) -> COLF
- U1 pad 34: unconnected-(U1-Pad34) -> COL0
- U1 pad 35: unconnected-(U1-Pad35) -> COL1
- U1 pad 36: unconnected-(U1-Pad36) -> COL2
- U1 pad 37: unconnected-(U1-Pad37) -> ROW2
- U1 pad 38: unconnected-(U1-Pad38) -> COL3
- U1 pad 39: unconnected-(U1-Pad39) -> COL4
- U1 pad 40: unconnected-(U1-Pad40) -> COL5
- U1 pad 41: unconnected-(U1-Pad41) -> ROW3
- U1 pad 6: unconnected-(U1-Pad6) -> ENC_B1
- U1 pad 7: unconnected-(U1-Pad7) -> ENC_A
Routing:
- net VCC: track 0.00 -> 1280.9 mm, vias 0 -> 15
- net ROW3: track 0.00 -> 459.1 mm, vias 0 -> 13
- net ROW2: track 0.00 -> 376.0 mm, vias 0 -> 2
- net ROW0: track 0.00 -> 362.8 mm, vias 0 -> 1
- net ROW1: track 0.00 -> 336.9 mm, vias 0 -> 4
- net COL0: track 0.00 -> 227.6 mm, vias 0 -> 2
- net COLF: track 0.00 -> 201.7 mm, vias 0 -> 3
- net COL1: track 0.00 -> 194.5 mm, vias 0 -> 2
- net COL6: track 0.00 -> 187.1 mm, vias 0 -> 2
- net COL7: track 0.00 -> 185.3 mm, vias 0 -> 2
- net COLE: track 0.00 -> 182.4 mm, vias 0 -> 3
- net Net-(DL1-Pad2): track 0.00 -> 173.6 mm, vias 0 -> 1
- net Net-(DL2-Pad2): track 0.00 -> 172.4 mm, vias 0 -> 1
- net RST: track 0.00 -> 171.7 mm, vias 0 -> 1
- net COL2: track 0.00 -> 169.7 mm, vias 0 -> 2
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