File: overboard.kicad_pcb (KiCad board)
At the start: 2 copper layers, 285 x 95.1 mm, 188 parts, among them J1 HRO-TYPE-C-31-M-12, J2 Conn_01x04, J3 Trackpoint, J4 Conn_01x04, J5 Conn_01x04, K00 Key_Switch, K01 Key_Switch, K02 Key_Switch, K03 Key_Switch, K10 Key_Switch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

Commit message: v0
Parts:
- added Ref**: Val**, User:Seal_Logo_12mm, F.Cu at (0.00, -14.3)
- moved LS1 40.9 mm to (67.9, -41.7)
Routing:
- net AUDIO: track 76.0 -> 107.4 mm
Other:
- board text added: "@t33chong"
- board text added: "JLCJLCJLCJLC"
- board text added: "Overboard v0"
