File: plate.kicad_pcb (KiCad board)
At the start: 2 copper layers, 285.4 x 94.9 mm, 74 parts, among them J10 Conn_01x02, J11 Conn_01x02, J8 Conn_01x02, J9 Conn_01x02, K00 MX_cutout, K01 MX_cutout, K02 MX_cutout, K03 MX_cutout, K10 MX_cutout, K11 MX_cutout, K12 MX_cutout, K13 MX_cutout, K20 MX_cutout, K21 MX_cutout, K22 MX_cutout, K23 MX_cutout, K30 MX_cutout, K31 MX_cutout, K32 MX_cutout, K33 MX_cutout, K40 MX_cutout, K41 MX_cutout, K42 MX_cutout, K43 MX_cutout, K50 MX_cutout, K51 MX_cutout, K52 MX_cutout, K53 MX_cutout, K92 MX_cutout, K93 MX_cutout, K94 MX_cutout

Commit message: Place components
Parts:
- removed J10, J11: Conn_01x02, Connector_PinHeader_2.54mm:PinHeader_1x02_P2.54mm_Vertical_SMD_Pin1Right
- added ENC1: Panasonic_EVQ-WGD001_Plate_Edge_Cuts, User:Panasonic_EVQ-WGD001_Plate_Edge_Cuts, F.Cu at (-11.9, 19.0)
- added ENC2: Panasonic_EVQ-WGD001_Plate_Edge_Cuts, User:Panasonic_EVQ-WGD001_Plate_Edge_Cuts, F.Cu at (11.9, 19.0)
- added OLED1: 128x64OLED_Edge_Cuts, User:128x64OLED_Edge_Cuts, F.Cu at (0.00, -33.2)
- added svg2mod: G***, User:Trackpoint_Outline, F.Cu at (0.00, 2.60)
- D60, D61, D62, D63, D64, D70, D71, D72, D73, D80, D81, D82, D83, D84: moved to B.Cu
- J4: renamed from J8; footprint Connector_PinHeader_2.54mm:PinHeader_1x02_P2.54mm_Vertical_SMD_Pin1Right -> Connector_PinHeader_2.54mm:PinHeader_1x04_P2.54mm_Vertical_SMD_Pin1Right; moved to B.Cu
- J5: renamed from J9; footprint Connector_PinHeader_2.54mm:PinHeader_1x02_P2.54mm_Vertical_SMD_Pin1Right -> Connector_PinHeader_2.54mm:PinHeader_1x04_P2.54mm_Vertical_SMD_Pin1Right; moved to B.Cu
- moved J4 255.1 mm to (-138.5, -22.2), turned to 180 degrees
- moved D61 232.9 mm to (-69.8, -41.3), turned to -90 degrees
- moved D60 226.4 mm to (-73.8, -41.3), turned to -90 degrees
- moved D62 225.9 mm to (-65.9, -41.3), turned to -90 degrees
- moved D70 218.1 mm to (-54.0, -41.3), turned to -90 degrees
- moved D64 213.9 mm to (-57.9, -41.3), turned to -90 degrees
- moved D63 212.5 mm to (-61.9, -41.3), turned to -90 degrees
- moved D71 208.4 mm to (-50.0, -41.3), turned to -90 degrees
- moved D72 149.3 mm to (50.0, -41.3), turned to -90 degrees
- moved NAV1 143.1 mm to (-14.0, -8.80), turned to -45 degrees
- moved D81 141.7 mm to (61.9, -41.3), turned to -90 degrees
- moved D73 136.1 mm to (54.0, -41.3), turned to -90 degrees
- moved D82 134.6 mm to (65.9, -41.3), turned to -90 degrees
- moved D83 130.8 mm to (69.8, -41.3), turned to -90 degrees
- moved D80 130.7 mm to (57.9, -41.3), turned to -90 degrees
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
Commit message: Route PCB & plate
Parts:
- removed the svg2mod at (0.00, 2.60)
- J4, J5: value Conn_01x02 -> Conn_01x04
- moved D64 101.7 mm to (43.7, -37.7)
- moved D61 101.6 mm to (31.8, -39.7)
- moved D82 97.7 mm to (-31.8, -39.3)
- moved D72 85.7 mm to (-35.7, -39.3)
- moved D71 85.7 mm to (35.7, -39.7)
- moved D63 81.8 mm to (19.8, -41.7)
- moved D80 77.8 mm to (-19.8, -41.7)
- moved D60 46.0 mm to (-27.8, -41.7)
- moved D83 42.1 mm to (27.8, -41.7)
- moved D70 30.2 mm to (-23.8, -41.7)
- moved D73 30.2 mm to (23.8, -41.7)
- moved D84 26.4 mm to (47.6, -37.7)
- moved D62 26.3 mm to (-39.7, -39.3)
- moved D81 22.3 mm to (39.7, -39.7)
Connections:
- J4 pad 2: COL6 -> ROW2
- J4 pad 3: (no net) -> COL6
- J4 pad 4: (no net) -> COL7
- J5 pad 1: ROW2 -> ROW1
- J5 pad 2: COL7 -> ROW3
- J5 pad 3: (no net) -> ROW4
- J5 pad 4: (no net) -> COL8
Routing:
- net COL7: track 0.00 -> 170.1 mm
- net COL8: track 0.00 -> 146.7 mm, vias 0 -> 1
- net COL6: track 0.00 -> 136.5 mm, vias 0 -> 1
- net ROW3: track 0.00 -> 134.2 mm
- net ROW0: track 0.00 -> 131.7 mm
- net ROW2: track 0.00 -> 119.7 mm
- net ROW1: track 0.00 -> 117.2 mm
- net ROW4: track 0.00 -> 110.1 mm
- net Net-(D64-Pad2): track 0.00 -> 91.9 mm, vias 0 -> 3
- net Net-(D61-Pad2): track 0.00 -> 75.3 mm, vias 0 -> 1
- net Net-(D82-Pad2): track 0.00 -> 61.8 mm, vias 0 -> 1
- net Net-(D84-Pad2): track 0.00 -> 56.6 mm, vias 0 -> 1
- net Net-(D70-Pad2): track 0.00 -> 56.0 mm
- net Net-(D60-Pad2): track 0.00 -> 54.9 mm, vias 0 -> 1
- net Net-(D71-Pad2): track 0.00 -> 53.6 mm, vias 0 -> 1
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
Commit message: v0
Parts:
- removed K01, K02, K11, KE1, KF1, KF2: MX_cutout, libmodulo:MX_cutout
- removed the svg2mod at (0.00, 0.00)
- added Ref**: Val**, User:Seal_Logo_12mm, B.Cu at (135.5, 40.2)
- added svg2mod: G***, User:Overboard_Plate, F.Cu at (0.00, 0.00)
- DIP1: footprint DS04-254-1L-04BK:SW_DS04-254-1L-04BK -> User:SW_DS04-254-1L-04BK
- NAV1, NAV2: value JOYSTICK_MINI -> >VALUE; footprint Sparkfun_Switches:JOYSTICK_MINI -> User:JOYSTICK_MINI
Routing:
- net Net-(D81-Pad2): track 51.9 -> 57.6 mm
- net Net-(D61-Pad2): track 75.3 -> 79.5 mm
- net Net-(D71-Pad2): track 53.6 -> 51.0 mm
- net Net-(D60-Pad2): track 54.9 -> 56.8 mm
- net COL8: track 146.7 -> 148.3 mm
- net Net-(D84-Pad2): track 56.6 -> 58.1 mm
- net ROW4: track 110.1 -> 111.3 mm
- net ROW1: track 117.2 -> 118.4 mm
- net Net-(D83-Pad2): track 37.9 -> 38.9 mm
- net ROW3: track 134.2 -> 135.1 mm
- net Net-(D64-Pad2): track 91.9 -> 92.8 mm
- net ROW2: track 119.7 -> 120.5 mm
- net ROW0: track 131.7 -> 132.3 mm
- net Net-(D70-Pad2): track 56.0 -> 56.6 mm
- net Net-(D62-Pad2): track 50.5 -> 51.1 mm
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Other:
- outline, holes or cut-outs redrawn
- board text added: "JLCJLCJLCJLC"
