File: plate.kicad_sch (KiCad schematic)
At the start: 26 parts, among them J10 Conn_01x02, J11 Conn_01x02, J8 Conn_01x02, J9 Conn_01x02

Commit message: Add plate, place RGB LEDs
Parts:
- removed H5, H6: MountingHole, User:MountingHole_5.3mm_M5, symbol Mechanical:MountingHole
- removed H7, H8: MountingHole, User:Montsinger_Side_Hole, symbol Mechanical:MountingHole
- D60, D61, D62, D63, D64, D70, D71, D72, D73, D80, D81, D82, D83, D84: value 1N4148 -> (none); footprint Diode_SMD:D_SOD-123 -> (none)
- DIP1: value DS04-254-1L-04BK -> (none); footprint DS04-254-1L-04BK:SW_DS04-254-1L-04BK -> (none)
- H1: renamed from H9; value MountingHole -> (none); footprint User:Trackpoint_Mounting_Holes -> (none)
- J10, J11, J8, J9: value Conn_01x02 -> (none); footprint Connector_PinHeader_2.54mm:PinHeader_1x02_P2.54mm_Vertical_SMD_Pin1Right -> (none)
- NAV1, NAV2: value JOYSTICK_MINI -> (none); footprint Sparkfun_Switches:JOYSTICK_MINI -> (none)

Commit message: Place components
Parts:
- removed J10, J11, J8, J9: (no value), symbol Connector_Generic:Conn_01x02
- added J4, J5: Conn_01x04, User:PinHeader_1x04_P2.54mm_Vertical_Centered, symbol Connector_Generic:Conn_01x04
- D60, D61, D62, D63, D64, D70, D71, D72, D73, D80, D81, D82, D83, D84: value (none) -> 1N4148; footprint (none) -> Diode_SMD:D_SOD-123
- DIP1: value (none) -> DS04-254-1L-04BK; footprint (none) -> DS04-254-1L-04BK:SW_DS04-254-1L-04BK
- H1: value (none) -> MountingHole; footprint (none) -> User:Trackpoint_Mounting_Holes
- NAV1, NAV2: value (none) -> JOYSTICK_MINI; footprint (none) -> Sparkfun_Switches:JOYSTICK_MINI
Connections:
- net COL6: now also J4.3 (Pin_3)
- net COL7: now also J4.4 (Pin_4)
- net COL8: now also J5.4 (Pin_4)
- net ROW0: now also J4.1 (Pin_1)
- net ROW1: now also J5.1 (Pin_1)
- net ROW2: now also J4.2 (Pin_2)
- net ROW3: now also J5.2 (Pin_2)
- net ROW4: now also J5.3 (Pin_3)
Other:
- moved on the sheet: H1

Commit message: Route PCB & plate
Parts:
- J4, J5: footprint User:PinHeader_1x04_P2.54mm_Vertical_Centered -> (none)
Changed lines of the file:
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@@
       (effects (font (size 1.27 1.27)) (justify left))
     )
-    (property "Footprint" "User:PinHeader_1x04_P2.54mm_Vertical_Centered" (id 2) (at 114.935 78.74 0)
+    (property "Footprint" "" (id 2) (at 114.935 78.74 0)
       (effects (font (size 1.27 1.27)) hide)
     )
@@
       (effects (font (size 1.27 1.27)) (justify left))
     )
-    (property "Footprint" "User:PinHeader_1x04_P2.54mm_Vertical_Centered" (id 2) (at 83.185 78.74 0)
+    (property "Footprint" "" (id 2) (at 83.185 78.74 0)
       (effects (font (size 1.27 1.27)) hide)
     )
@@
     )
     (path "/199f157d-6f84-41da-be4c-6e21ffdc4f00"
-      (reference "J4") (unit 1) (value "Conn_01x04") (footprint "User:PinHeader_1x04_P2.54mm_Vertical_Centered")
+      (reference "J4") (unit 1) (value "Conn_01x04") (footprint "Connector_PinHeader_2.54mm:PinHeader_1x04_P2.54mm_Vertical_SMD_Pin1Right")
     )
     (path "/05a3fd88-c58e-4323-96ff-70847ec682b8"
-      (reference "J5") (unit 1) (value "Conn_01x04") (footprint "User:PinHeader_1x04_P2.54mm_Vertical_Centered")
+      (reference "J5") (unit 1) (value "Conn_01x04") (footprint "Connector_PinHeader_2.54mm:PinHeader_1x04_P2.54mm_Vertical_SMD_Pin1Right")
     )
     (path "/7e623bc6-23b6-4661-93b8-1f672e1d4d74"

Commit message: v0
Parts:
- DIP1: footprint DS04-254-1L-04BK:SW_DS04-254-1L-04BK -> (none)
- J4, J5: footprint (none) -> Connector_PinHeader_2.54mm:PinHeader_1x04_P2.54mm_Vertical_SMD_Pin1Right
- NAV1, NAV2: footprint Sparkfun_Switches:JOYSTICK_MINI -> (none)
Changed lines of the file:
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@@
       (effects (font (size 1.27 1.27)) (justify left))
     )
-    (property "Footprint" "" (id 2) (at 114.935 78.74 0)
+    (property "Footprint" "Connector_PinHeader_2.54mm:PinHeader_1x04_P2.54mm_Vertical_SMD_Pin1Right" (id 2) (at 114.935 78.74 0)
       (effects (font (size 1.27 1.27)) hide)
     )
@@
       (effects (font (size 1.27 1.27)) (justify left))
     )
-    (property "Footprint" "" (id 2) (at 83.185 78.74 0)
+    (property "Footprint" "Connector_PinHeader_2.54mm:PinHeader_1x04_P2.54mm_Vertical_SMD_Pin1Right" (id 2) (at 83.185 78.74 0)
       (effects (font (size 1.27 1.27)) hide)
     )
@@
       (effects (font (size 1.143 1.143)))
     )
-    (property "Footprint" "Sparkfun_Switches:JOYSTICK_MINI" (id 2) (at 233.045 32.385 0)
+    (property "Footprint" "" (id 2) (at 233.045 32.385 0)
       (effects (font (size 0.508 0.508)) hide)
     )
@@
       (effects (font (size 1.143 1.143)))
     )
-    (property "Footprint" "Sparkfun_Switches:JOYSTICK_MINI" (id 2) (at 54.61 32.385 0)
+    (property "Footprint" "" (id 2) (at 54.61 32.385 0)
       (effects (font (size 0.508 0.508)) hide)
     )
@@
     (property "Reference" "DIP1" (id 0) (at 133.985 25.4 0))
     (property "Value" "DS04-254-1L-04BK" (id 1) (at 133.985 27.94 0))
-    (property "Footprint" "DS04-254-1L-04BK:SW_DS04-254-1L-04BK" (id 2) (at 133.985 40.64 0)
+    (property "Footprint" "" (id 2) (at 133.985 40.64 0)
       (effects (font (size 1.27 1.27)) (justify left bottom) hide)
     )
@@
     )
     (path "/f8bbaa62-8626-4601-bf34-80d8fe5e6f74"
-      (reference "DIP1") (unit 1) (value "DS04-254-1L-04BK") (footprint "DS04-254-1L-04BK:SW_DS04-254-1L-04BK")
+      (reference "DIP1") (unit 1) (value "DS04-254-1L-04BK") (footprint "User:SW_DS04-254-1L-04BK")
     )
     (path "/8f2140d1-7e63-42c6-b5a9-2853a8966a28"
@@
     )
     (path "/7e623bc6-23b6-4661-93b8-1f672e1d4d74"
-      (reference "NAV1") (unit 1) (value "JOYSTICK_MINI") (footprint "Sparkfun_Switches:JOYSTICK_MINI")
+      (reference "NAV1") (unit 1) (value "JOYSTICK_MINI") (footprint "User:JOYSTICK_MINI")
     )
     (path "/27f35f65-af8e-49b7-95d2-ba17e14c608c"
-      (reference "NAV2") (unit 1) (value "JOYSTICK_MINI") (footprint "Sparkfun_Switches:JOYSTICK_MINI")
-    )
-  )
+      (reference "NAV2") (unit 1) (value "JOYSTICK_MINI") (footprint "User:JOYSTICK_MINI")
+    )
+  )
